File: Locomotive/Locomotive.sch (KiCad schematic (older format))
At the start: 4 parts

Commit message: Add & Align Pins
Add pins to all trains and set proper locations
Move RGB LEDs and resistors
Connect RGB LEDs to resistors and speaker to Arduino
Parts:
- MK2: value 2 -> GND
Connections:
- net labels added: GND, VCC
Changed lines of the file:
@@
 P 3375 4825
 F 0 "MK2" H 3275 4783 50  0000 R CNN
-F 1 "2" H 3275 4874 50  0000 R CNN
+F 1 "GND" H 3275 4874 50  0000 R CNN
 F 2 "Pin_Headers:Pin_Header_Angled_1x01_Pitch2.54mm" H 3375 4825 50  0001 C CNN
 F 3 "" H 3375 4825 50  0001 C CNN
@@
 Wire Wire Line
 	3375 4350 3375 4725
+Text Label 2375 4550 0    50   ~ 0
+VCC
+Text Label 3375 4625 0    50   ~ 0
+GND
 $EndSCHEMATC
