File: Boxcar/Boxcar.sch (KiCad schematic (older format))
At the start: 6 parts

Commit message: Change Schematic For RGB LEDs
Add transistors to control 3 RGB LEDs
Add Silkscreen detail to caboose
Parts:
- D1, D2: footprint LEDs:LED_1206_HandSoldering -> LEDs:LED_0805_HandSoldering
Changed lines of the file:
@@
 F 0 "D1" H 2892 2845 50  0000 C CNN
 F 1 "LED" H 2892 2936 50  0000 C CNN
-F 2 "LEDs:LED_1206_HandSoldering" H 2900 3100 50  0001 C CNN
+F 2 "LEDs:LED_0805_HandSoldering" H 2900 3100 50  0001 C CNN
 F 3 "~" H 2900 3100 50  0001 C CNN
 	1    2900 3100
@@
 F 0 "D2" H 3167 3320 50  0000 C CNN
 F 1 "LED" H 3167 3411 50  0000 C CNN
-F 2 "LEDs:LED_1206_HandSoldering" H 3175 3575 50  0001 C CNN
+F 2 "LEDs:LED_0805_HandSoldering" H 3175 3575 50  0001 C CNN
 F 3 "~" H 3175 3575 50  0001 C CNN
 	1    3175 3575
