File: Boxcar/Boxcar.kicad_pcb (KiCad board)
At the start: 2 copper layers, 47.5 x 16.5 mm, 8 parts

Commit message: Update Text
Change dates on trains
Other:
- board text added: "100Ω"
Changed lines of the file:
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@@
-(kicad_pcb (version 20171130) (host pcbnew 5.0.0-rc2-dev-unknown-2bab30d~65~ubuntu16.04.1)
+(kicad_pcb (version 20171130) (host pcbnew 5.0.0-rc2-dev-unknown-d09445c~65~ubuntu16.04.1)
   (general
     (thickness 1.6)
-    (drawings 1486)
+    (drawings 1488)
     (tracks 11)
     (zones 0)
@@
     (visible_elements FFFFFF7F)
     (pcbplotparams
-      (layerselection 0x010fc_ffffffff)
-      (usegerberextensions false)
+      (layerselection 0x010f0_ffffffff)
+      (usegerberextensions true)
       (usegerberattributes false)
       (usegerberadvancedattributes false)
@@
       (outputformat 1)
       (mirror false)
-      (drillshape 1)
+      (drillshape 0)
       (scaleselection 1)
-      (outputdirectory ""))
+      (outputdirectory GERBER/))
   )
   (net 0 "")
@@
     (tags "resistor 1206")
     (attr smd)
-    (fp_text reference R1 (at 0 1.85) (layer B.SilkS)
+    (fp_text reference R1 (at 0 1.85) (layer B.Fab)
       (effects (font (size 1 1) (thickness 0.15)) (justify mirror))
     )
@@
     (tags "resistor 1206")
     (attr smd)
-    (fp_text reference R2 (at 0 1.85) (layer B.SilkS)
+    (fp_text reference R2 (at 0 1.85) (layer B.Fab)
       (effects (font (size 1 1) (thickness 0.15)) (justify mirror))
     )
@@
     )
   )
+  (gr_text 100Ω (at 27.305 57.15) (layer B.SilkS)
+    (effects (font (size 1 1) (thickness 0.25)) (justify mirror))
+  )
+  (gr_text 100Ω (at 14.732 57.15) (layer B.SilkS)
+    (effects (font (size 1 1) (thickness 0.25)) (justify mirror))
+  )
   (gr_line (start 0.466751 61.980734) (end 0.458561 61.978588) (layer Edge.Cuts) (width 0.15))
