File: Caboose/Caboose.sch (KiCad schematic (older format))
At the start: 6 parts

Commit message: Change Schematic For RGB LEDs
Add transistors to control 3 RGB LEDs
Add Silkscreen detail to caboose
Parts:
- D1, D2: footprint LEDs:LED_1206_HandSoldering -> LEDs:LED_0805_HandSoldering
Changed lines of the file:
@@
 F 0 "D1" H 2592 2845 50  0000 C CNN
 F 1 "LED" H 2592 2936 50  0000 C CNN
-F 2 "LEDs:LED_1206_HandSoldering" H 2600 3100 50  0001 C CNN
+F 2 "LEDs:LED_0805_HandSoldering" H 2600 3100 50  0001 C CNN
 F 3 "~" H 2600 3100 50  0001 C CNN
 	1    2600 3100
@@
 F 0 "D2" H 2567 3320 50  0000 C CNN
 F 1 "LED" H 2567 3411 50  0000 C CNN
-F 2 "LEDs:LED_1206_HandSoldering" H 2575 3575 50  0001 C CNN
+F 2 "LEDs:LED_0805_HandSoldering" H 2575 3575 50  0001 C CNN
 F 3 "~" H 2575 3575 50  0001 C CNN
 	1    2575 3575
